File: sensorBoardMk2.kicad_pcb (KiCad board)
At the start: 2 copper layers, 63 x 63 mm, 50 parts, among them J1 S4B-PH-K-S__LF__SN_, J2 S4B-PH-K-S__LF__SN_, P1 TP, P2 TP, P3 TP, P4 TP, P5 TP, U1 SHT45, U2 BME280, U3 SGP40-D-R4

Commit message: Made the damn thing smaller
Parts:
- removed the G*** at (44.8, 77.0)
- removed the G*** at (71.2, 98.4)
- removed the G*** at (35.0, 69.6)
- removed the G*** at (26.2, 67.0)
- removed the G*** at (27.0, 97.4)
- moved D6 30.0 mm to (45.1, 68.0)
- moved R4 30.0 mm to (45.1, 63.8)
- moved J2 21.4 mm to (75.4, 24.0)
- moved MountingHoleBottom 20.7 mm to (46.7, 77.0)
- moved MountingHoleTop 20.7 mm to (46.7, 26.0)
- moved G*** 19.6 mm to (55.1, 73.4)
- moved J1 17.5 mm to (56.5, 24.0)
- moved C5 17.3 mm to (47.5, 55.3), turned to 0 degrees
- moved JP1 16.4 mm to (52.1, 51.4), turned to 90 degrees
- moved C6 13.9 mm to (47.5, 52.7), turned to 0 degrees
- moved C9 12.0 mm to (56.6, 55.5)
- moved P1 10.5 mm to (52.2, 37.2)
- moved R2 10.5 mm to (48.2, 37.2)
- moved P2 10.5 mm to (55.4, 37.2)
- moved R1 10.5 mm to (59.4, 37.2)
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Routing:
- net +3.3V: track 162.7 -> 148.2 mm
- net /ADC: track 65.6 -> 74.0 mm, vias 0 -> 2
- net /INT: track 74.8 -> 68.3 mm, vias 2 -> 0
- net /SCL: track 50.8 -> 45.2 mm, vias 3 -> 0
- net /SDA: track 49.0 -> 53.4 mm, vias 0 -> 3
Other:
- board size 63 x 63 mm -> 42.3 x 63 mm

Commit message: Did some improvements based on feedback from lil brother
Parts:
- moved C3 0.11 mm to (49.1, 33.5)
Connections:
- MountingHoleBottom pad 1: (no net) -> GND
- MountingHoleTop pad 1: (no net) -> GND
Routing:
- net GND: track 44.7 -> 4.26 mm, vias 12 -> 17
- net +3.3V: track 148.2 -> 146.5 mm, vias 4 -> 9
- added copper zone on F.Cu, net GND
